Commit message: Working on making the camera position publish correctly using Aruco as known position

File: simulation/src/sim/urdf/my_robot_tf.urdf (robot description, URDF)
Before this commit: robot my_robot, 5 links, 4 joints
Links:
- removed link odom
- added link zed2i_left_optical_frame
Joints:
- removed joint odom_to_base_link
- added joint zed2i_optical_joint: type fixed, parent zed2i_base_link, child zed2i_left_optical_frame, origin xyz=0 0 0 rpy=-1.5708 0 -1.5708
