Commit message: Modified launch files

File: shovel/src/sim/urdf/my_robot_tf.urdf (robot description, URDF)
Before this commit: robot my_robot, 13 links, 12 joints
Joints:
- joint BL_Wheel_Joint: origin xyz=0.18387 0 0.23588 rpy=0 0 0 -> xyz=0.18387 0 0.23588 rpy=1.5708 0 0
- joint BR_Wheel_Joint: origin xyz=0.183875 -0.475667 0.235883 rpy=0 0 -3.14159 -> xyz=0.183875 -0.475667 0.235883 rpy=1.5708 0 -3.14159
- joint FL_Wheel_Joint: origin xyz=0.8411 -0.019814 0.235883 rpy=0 0 0 -> xyz=0.8411 -0.019814 0.235883 rpy=1.5708 0 0
- joint FR_Wheel_Joint: origin xyz=0.8411 -0.538167 0.235883 rpy=0 0 0 -> xyz=0.8411 -0.538167 0.235883 rpy=1.5708 0 0
- joint base_to_d455i: origin xyz=0 0 0 rpy=0 0 0 -> xyz=0.85 -0.55 0.5 rpy=0 0.35 0

Commit message: Working on things

File: shovel/src/sim/urdf/my_robot_tf.urdf (robot description, URDF)
Before this commit: robot my_robot, 13 links, 12 joints
Links:
- added link zed2i_right_optical_frame
Joints:
- removed joint zed2i_optical_joint
- added joint zed2i_left_optical_joint: type fixed, parent zed2i_base_link, child zed2i_left_optical_frame, origin xyz=0 -0.06 0 rpy=-1.5708 0 -1.5708
- added joint zed2i_right_optical_joint: type fixed, parent zed2i_base_link, child zed2i_right_optical_frame, origin xyz=0 0.06 0 rpy=-1.5708 0 -1.5708
- joint BL_Wheel_Joint: axis 0 0 -1 -> 0 1 0; origin xyz=0.18387 0 0.23588 rpy=1.5708 0 0 -> xyz=0.18387 0 0.23588 rpy=0 0 0
- joint BR_Wheel_Joint: axis 0 0 1 -> 0 -1 0; origin xyz=0.183875 -0.475667 0.235883 rpy=1.5708 0 -3.14159 -> xyz=0.183875 -0.475667 0.235883 rpy=0 0 -3.14159
- joint FL_Wheel_Joint: axis 0 0 -1 -> 0 1 0; origin xyz=0.8411 -0.019814 0.235883 rpy=1.5708 0 0 -> xyz=0.8411 -0.019814 0.235883 rpy=0 0 0
- joint FR_Wheel_Joint: axis 0 0 -1 -> 0 1 0; origin xyz=0.8411 -0.538167 0.235883 rpy=1.5708 0 0 -> xyz=0.8411 -0.538167 0.235883 rpy=0 0 0
- joint d455i_to_lidar: origin xyz=0 0 0 rpy=0 0 0 -> xyz=0 0 0.2 rpy=0 0 0
